File: board/board.kicad_pcb (KiCad board)
At the start: 2 copper layers, 21 x 13 mm, 1 part

Commit message: initial
Parts:
- added U1: BK-6223-TR, b117:AAA_cell_holder, F.Cu at (172.4, 115.5)
- added U2: BK-6223-TR, b117:AAA_cell_holder, F.Cu at (172.4, 126.0)
Other:
- board size 21 x 13 mm -> 46 x 9 mm
Changed lines of the file:
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@@
   )
   (net 0 "")
+  (net 1 "/2x_aaa/Low")
+  (net 2 "/2x_aaa/Mid")
+  (net 3 "/2x_aaa/High")
   (footprint "Symbol:OSHW-Symbol_6.7x6mm_SilkScreen" (layer "F.Cu")
     (at 150 99)
@@
       ) (layer "F.SilkS") (width 0.01) (fill solid))
   )
+  (footprint "b117:AAA_cell_holder" (layer "F.Cu")
+    (at 172.4 115.5)
+    (property "Sheetfile" "2x_aaa.kicad_sch")
+    (property "Sheetname" "2x_aaa")
+    (fp_text reference "U1" (at 0 -0.5 unlocked) (layer "F.SilkS")
+      (effects (font (size 1 1) (thickness 0.15)))
+    )
+    (fp_text value "BK-6223-TR" (at 0 1 unlocked) (layer "F.Fab")
+      (effects (font (size 1 1) (thickness 0.15)))
+    )
+    (fp_text user "${REFERENCE}" (at 0 2.5 unlocked) (layer "F.Fab")
+      (effects (font (size 1 1) (thickness 0.15)))
+    )
+    (fp_line (start 23.2 4.7) (end 23.2 -4.7) (layer "F.SilkS") (width 0.12))
+    (fp_line (start 23.2 -4.7) (end -23.2 -4.7) (layer "F.SilkS") (width 0.12))
+    (fp_line (start -23.2 4.7) (end 23.2 4.7) (layer "F.SilkS") (width 0.12))
+    (fp_line (start -23.2 -4.7) (end -23.2 4.7) (layer "F.SilkS") (width 0.12))
+    (fp_line (start -23 -4.5) (end -23 4.5) (layer "Edge.Cuts") (width 0.12))
+    (fp_line (start 23 4.5) (end 23 -4.5) (layer "Edge.Cuts") (width 0.12))
+    (fp_line (start 23 -4.5) (end -23 -4.5) (layer "Edge.Cuts") (width 0.12))
+    (fp_line (start -23 4.5) (end 23 4.5) (layer "Edge.Cuts") (width 0.12))
+    (pad "1" thru_hole rect (at -27.5 0) (size 6 6) (drill 0.762) (layers *.Cu *.Mask)
+      (net 1 "/2x_aaa/Low") (pintype "unspecified"))
+    (pad "2" thru_hole rect (at 27.5 0) (size 6 6) (drill 0.762) (layers *.Cu *.Mask)
+      (net 2 "/2x_aaa/Mid") (pintype "unspecified"))
+    (model "${KIPRJMOD}/b117.pretty/AAA battery.stp"
+      (offset (xyz 82.5 -64 2.5))
+      (scale (xyz 1 1 1))
+      (rotate (xyz 0 0 -90))
+    )
+  )
+  (footprint "b117:AAA_cell_holder" (layer "F.Cu")
+    (at 172.4 126.02)
+    (property "Sheetfile" "2x_aaa.kicad_sch")
+    (property "Sheetname" "2x_aaa")
+    (fp_text reference "U2" (at 0 -0.5 unlocked) (layer "F.SilkS")
+      (effects (font (size 1 1) (thickness 0.15)))
+    )
+    (fp_text value "BK-6223-TR" (at 0 1 unlocked) (layer "F.Fab")
+      (effects (font (size 1 1) (thickness 0.15)))
+    )
+    (fp_text user "${REFERENCE}" (at 0 2.5 unlocked) (layer "F.Fab")
+      (effects (font (size 1 1) (thickness 0.15)))
+    )
+    (fp_line (start 23.2 -4.7) (end -23.2 -4.7) (layer "F.SilkS") (width 0.12))
+    (fp_line (start -23.2 -4.7) (end -23.2 4.7) (layer "F.SilkS") (width 0.12))
+    (fp_line (start 23.2 4.7) (end 23.2 -4.7) (layer "F.SilkS") (width 0.12))
+    (fp_line (start -23.2 4.7) (end 23.2 4.7) (layer "F.SilkS") (width 0.12))
+    (fp_line (start 23 -4.5) (end -23 -4.5) (layer "Edge.Cuts") (width 0.12))
+    (fp_line (start 23 4.5) (end 23 -4.5) (layer "Edge.Cuts") (width 0.12))
+    (fp_line (start -23 4.5) (end 23 4.5) (layer "Edge.Cuts") (width 0.12))
+    (fp_line (start -23 -4.5) (end -23 4.5) (layer "Edge.Cuts") (width 0.12))
+    (pad "1" thru_hole rect (at -27.5 0) (size 6 6) (drill 0.762) (layers *.Cu *.Mask)
+      (net 2 "/2x_aaa/Mid") (pintype "unspecified"))
+    (pad "2" thru_hole rect (at 27.5 0) (size 6 6) (drill 0.762) (layers *.Cu *.Mask)
+      (net 3 "/2x_aaa/High") (pintype "unspecified"))
+    (model "${KIPRJMOD}/b117.pretty/AAA battery.stp"
+      (offset (xyz 82.5 -64 2.5))
+      (scale (xyz 1 1 1))
+      (rotate (xyz 0 0 -90))
+    )
+  )
   (gr_line (start 142 90) (end 159 90) (layer "Edge.Cuts") (width 0.05))
